File: HestiaPi-ONE/KiCAD/HestiaPiOneUniversal.kicad_sch (KiCad schematic)
At the start: 14 parts, among them J0 RPi_GPIO, J3 LCD_pins, J4 AC/N, J5 AC/L, J6 GND, J7 5V, SW1 PB400OAQR1BLK

Commit message: Version 2.54 of the PCB design (warning: has errors)
Parts:
- added RL5: RL4, Library:Panasonic_AQ-G_relay, symbol Panasonic_AQ-G_relay:Panasonic_AQ-G_relay
- J0: footprint rPi_Zero_Socketed_THT_FaceDown_MountingHoles -> Module:Raspberry_Pi_Zero_Socketed_THT_FaceDown_MountingHoles
- J3: Mouser link (none) -> https://www.mouser.com/ProductDetail/Samtec/MTSW-113-07-T-D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; Note (none) -> Pins are intentionally reversed because we go through a rib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; cable datasheet (none) -> https://www.mouser.com/datasheet/2/527/hcmd-2498159.pdf; cable mouser (none) -> https://www.mouser.com/ProductDetail/Samtec/HCMD-13-T-04.00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
- SW1: value PB400OAQR1BLK -> PB400EEQX; Mouser link https://www.mouser.com/ProductDetail/E-Switch/PB400OAQR1BLK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 -> https://www.mouser.com/ProductDetail/E-Switch/PB400EEQX?qs=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
- TerminalBlock1: renamed from C(N)  R(L)  W(W)  Y(H)  G(Hum)  W2; value Screw_Terminal_01x06 -> Screw_Terminal_01x07; footprint TerminalBlock_Phoenix:TerminalBlock_Phoenix_PT-1,5-6-5.0-H_1x06_P5.00mm_Horizontal -> TerminalBlock_Phoenix:TerminalBlock_Phoenix_PT-1,5-7-5.0-H_1x07_P5.00mm_Horizontal; symbol Connector:Screw_Terminal_01x06 -> Connector:Screw_Terminal_01x07
Connections:
- net A/C-L: now also RL5.2 (load2)
- net GND: now also J3.10 (Pin_10), J3.13 (Pin_13), J3.19 (Pin_19), J3.26 (Pin_26), J3.5 (Pin_5), RL5.4 (Input-); no longer J3.14 (Pin_14), J3.20 (Pin_20), J3.25 (Pin_25), J3.6 (Pin_6), J3.9 (Pin_9)
- net at J0.2 (5V), SW1.1 (A): now also J3.1 (Pin_1); no longer J3.2 (Pin_2)
- net Net-(TerminalBlock1-Pad1): now reaches J4.1 (Pin_1), PSU-EU_100-240V_AC1.2 (AC/N), TerminalBlock1.1 (Pin_1)
- net Net-(TerminalBlock1-Pad3): now reaches RL1.1 (load1), TerminalBlock1.3 (Pin_3)
- net Net-(TerminalBlock1-Pad4): now reaches RL2.1 (load1), TerminalBlock1.4 (Pin_4)
- net at J0.12 (GPIO18), RL3.3 (Input+): no longer J3.12 (Pin_12)
- net at J0.16 (GPIO23), RL2.3 (Input+): no longer J3.16 (Pin_16)
- net at BME280.4 (Pin_4), J0.1 (3.3V): now also J3.2 (Pin_2); no longer J3.1 (Pin_1)
- net at J0.10 (GPIO15_RXD0): now also J3.11 (Pin_11); no longer J3.10 (Pin_10)
- net at J0.11 (GPIO17): now also J3.12 (Pin_12); no longer J3.11 (Pin_11)
- net at J0.13 (GPIO27): no longer J3.13 (Pin_13)
- net at J3.15 (Pin_15): no longer J0.15 (GPIO22)
- net at J3.17 (Pin_17): now also J0.18 (GPIO24); no longer J0.17 (3.3V)
- net at J3.18 (Pin_18): now also J0.17 (3.3V); no longer J0.18 (GPIO24)
- net at J0.19 (GPIO10_SPI_MOSI): now also J3.20 (Pin_20); no longer J3.19 (Pin_19)
- net at J3.21 (Pin_21): now also J0.22 (GPIO25); no longer J0.21 (GPIO09_SPI_MISO)
- net at J3.22 (Pin_22): now also J0.21 (GPIO09_SPI_MISO); no longer J0.22 (GPIO25)
- net at J3.23 (Pin_23): now also J0.24 (GPIO08_SPI_CE0_N); no longer J0.23 (GPIO11_SPI_CLK)
- net at J3.24 (Pin_24): now also J0.23 (GPIO11_SPI_CLK); no longer J0.24 (GPIO08_SPI_CE0_N)
- net at J0.26 (GPIO07_SPI_CE1_N): now also J3.25 (Pin_25); no longer J3.26 (Pin_26)
- net at BME280.1 (Pin_1), J0.3 (GPIO02_SDA1_I2C): no longer J3.3 (Pin_3)
- net at J0.4 (5V): now also J3.3 (Pin_3); no longer J3.4 (Pin_4)
- net at BME280.2 (Pin_2), J0.5 (GPIO03_SCL1_I2C): no longer J3.5 (Pin_5)
- net at J3.7 (Pin_7): no longer J0.7 (GPIO04_GCLK)
- net at J3.8 (Pin_8): no longer J0.8 (GPIO14_TXD0)
- net Net-(J0-Pad36): now reaches J0.36 (GPIO16)
- net Net-(J0-Pad36): now also RL5.3 (Input+)
- new net Net-(TerminalBlock1-Pad7): RL5.1 (load1), TerminalBlock1.7 (Pin_7)
- no-connect marks 11 -> 22

Commit message: Version 2.55 of the PCB design (warning: has errors)
Connections:
- net A/C-L: no longer RL5.2 (load2)
- net GND: no longer RL5.4 (Input-)
- net Net-(TerminalBlock1-Pad7): no longer RL5.1 (load1)
- net at RL4.3 (Input+): now also J0.36 (GPIO16); no longer J0.38 (GPIO20)
- net Net-(J0-Pad36): no longer names the net of RL5.3 (Input+)
- net Net-(J0-Pad36): no longer J0.36 (GPIO16)
Changed lines of the file:
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@@
     (stroke (width 0) (type default) (color 0 0 0 0))
   )
-  (wire (pts (xy 228.6 95.25) (xy 228.6 91.44))
+  (wire (pts (xy 228.6 95.25) (xy 228.6 93.98))
     (stroke (width 0) (type default) (color 0 0 0 0))
   )
@@
     (stroke (width 0) (type default) (color 0 0 0 0))
   )
+  (wire (pts (xy 237.49 93.98) (xy 267.97 93.98))
+    (stroke (width 0) (type default) (color 0 0 0 0))
+  )
   (wire (pts (xy 92.71 78.74) (xy 92.71 138.43))
     (stroke (width 0) (type default) (color 0 0 0 0))
@@
     (stroke (width 0) (type default) (color 0 0 0 0))
   )
+  (wire (pts (xy 237.49 91.44) (xy 237.49 93.98))
+    (stroke (width 0) (type default) (color 0 0 0 0))
+  )
   (wire (pts (xy 201.93 50.8) (xy 201.93 58.42))
     (stroke (width 0) (type default) (color 0 0 0 0))
@@
     (stroke (width 0) (type default) (color 0 0 0 0))
   )
-  (wire (pts (xy 228.6 91.44) (xy 166.37 91.44))
-    (stroke (width 0) (type default) (color 0 0 0 0))
-  )
   (wire (pts (xy 265.43 90.17) (xy 265.43 97.79))
     (stroke (width 0) (type default) (color 0 0 0 0))
@@
     (stroke (width 0) (type default) (color 0 0 0 0))
   )
+  (wire (pts (xy 166.37 91.44) (xy 237.49 91.44))
+    (stroke (width 0) (type default) (color 0 0 0 0))
+  )
   (wire (pts (xy 196.85 67.31) (xy 205.74 67.31))
     (stroke (width 0) (type default) (color 0 0 0 0))
@@
     (stroke (width 0) (type default) (color 0 0 0 0))
   )
-  (wire (pts (xy 267.97 93.98) (xy 166.37 93.98))
-    (stroke (width 0) (type default) (color 0 0 0 0))
-  )
   (wire (pts (xy 104.14 48.26) (xy 104.14 27.94))
     (stroke (width 0) (type default) (color 0 0 0 0))
@@
     (stroke (width 0) (type default) (color 0 0 0 0))
   )
+  (wire (pts (xy 166.37 93.98) (xy 228.6 93.98))
+    (stroke (width 0) (type default) (color 0 0 0 0))
+  )
   (wire (pts (xy 265.43 81.28) (xy 265.43 77.47))
     (stroke (width 0) (type default) (color 0 0 0 0))
@@
   (wire (pts (xy 96.52 71.12) (xy 118.11 71.12))
     (stroke (width 0) (type default) (color 0 0 0 0))
-  )
-  (label "A{slash}C-L" (at 279.47 85.12 0)
-    (effects (font (size 1.27 1.27)) (justify left bottom))
   )
   (label "Net-(TerminalBlock1-Pad7)" (at 212.09 104.14 270)
     (effects (font (size 1.27 1.27)) (justify right bottom))
   )
-  (label "GND" (at 279.47 97.82 0)
-    (effects (font (size 1.27 1.27)) (justify left bottom))
-  )
-  (label "Net-(J0-Pad36)" (at 166.37 91.44 0)
-    (effects (font (size 1.27 1.27)) (justify left bottom))
-  )
   (label "Net-(TerminalBlock1-Pad4)" (at 204.47 104.14 270)
     (effects (font (size 1.27 1.27)) (justify right bottom))
@@
     (effects (font (size 1.27 1.27)) (justify right bottom))
   )
-  (label "Net-(J0-Pad36)" (at 279.47 95.28 0)
-    (effects (font (size 1.27 1.27)) (justify left bottom))
-  )
   (label "Net-(TerminalBlock1-Pad1)" (at 196.85 104.14 270)
     (effects (font (size 1.27 1.27)) (justify right bottom))
   )
-  (label "Net-(TerminalBlock1-Pad7)" (at 279.47 77.5 0)
-    (effects (font (size 1.27 1.27)) (justify left bottom))
-  )
   (global_label "A{slash}C-L" (shape input) (at 220.98 49.53 0) (fields_autoplaced)

Commit message: Version 2.56 of the PCB design (warning: not fully tested)
Parts:
- J4: value AC/N -> wire
- J5: value AC/L -> wire
- J6: value GND -> wire
- J7: value 5V -> wire
- RL1: value RL1 -> RL
- RL2: value RL2 -> RL
- RL3: value RL3 -> RL
- RL4, RL5: value RL4 -> RL
Changed lines of the file:
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@@
     (in_bom yes) (on_board yes) (fields_autoplaced)
     (property "Reference" "RL5" (id 0) (at 278.13 69.85 90))
-    (property "Value" "RL4" (id 1) (at 278.13 72.39 90))
+    (property "Value" "RL" (id 1) (at 278.13 72.39 90))
     (property "Footprint" "Library:Panasonic_AQ-G_relay" (id 2) (at 281.94 83.82 0)
       (effects (font (size 1.27 1.27)) hide)
@@
     (in_bom yes) (on_board yes) (fields_autoplaced)
     (property "Reference" "J5" (id 0) (at 192.405 53.34 0))
-    (property "Value" "AC/L" (id 1) (at 192.405 55.88 0))
+    (property "Value" "wire" (id 1) (at 192.405 55.88 0))
     (property "Footprint" "Connector_PinHeader_2.54mm:PinHeader_1x01_P2.54mm_Vertical" (id 2) (at 191.77 58.42 0)
       (effects (font (size 1.27 1.27)) hide)
@@
     (in_bom yes) (on_board yes) (fields_autoplaced)
     (property "Reference" "RL4" (id 0) (at 264.09 62.2 90))
-    (property "Value" "RL4" (id 1) (at 264.09 64.74 90))
+    (property "Value" "RL" (id 1) (at 264.09 64.74 90))
     (property "Footprint" "Library:Panasonic_AQ-G_relay" (id 2) (at 267.9 76.17 0)
       (effects (font (size 1.27 1.27)) hide)
@@
     (in_bom yes) (on_board yes)
     (property "Reference" "J6" (id 0) (at 172.085 26.67 0))
-    (property "Value" "GND" (id 1) (at 172.085 29.21 0))
+    (property "Value" "wire" (id 1) (at 172.085 29.21 0))
     (property "Footprint" "Connector_PinHeader_2.54mm:PinHeader_1x01_P2.54mm_Vertical" (id 2) (at 171.45 31.75 0)
       (effects (font (size 1.27 1.27)) hide)
@@
     (in_bom yes) (on_board yes) (fields_autoplaced)
     (property "Reference" "RL3" (id 0) (at 248.85 58.39 90))
-    (property "Value" "RL3" (id 1) (at 248.85 60.93 90))
+    (property "Value" "RL" (id 1) (at 248.85 60.93 90))
     (property "Footprint" "Library:Panasonic_AQ-G_relay" (id 2) (at 234.88 87.6 0)
       (effects (font (size 1.27 1.27)) hide)
@@
     (in_bom yes) (on_board yes) (fields_autoplaced)
     (property "Reference" "RL2" (id 0) (at 233.61 54.58 90))
-    (property "Value" "RL2" (id 1) (at 233.61 57.12 90))
+    (property "Value" "RL" (id 1) (at 233.61 57.12 90))
     (property "Footprint" "Library:Panasonic_AQ-G_relay" (id 2) (at 219.64 83.79 0)
       (effects (font (size 1.27 1.27)) hide)
@@
     (in_bom yes) (on_board yes) (fields_autoplaced)
     (property "Reference" "J7" (id 0) (at 180.975 54.61 0))
-    (property "Value" "5V" (id 1) (at 180.975 57.15 0))
+    (property "Value" "wire" (id 1) (at 180.975 57.15 0))
     (property "Footprint" "Connector_PinHeader_2.54mm:PinHeader_1x01_P2.54mm_Vertical" (id 2) (at 180.34 59.69 0)
       (effects (font (size 1.27 1.27)) hide)
@@
     (in_bom yes) (on_board yes) (fields_autoplaced)
     (property "Reference" "J4" (id 0) (at 197.485 35.56 0))
-    (property "Value" "AC/N" (id 1) (at 197.485 38.1 0))
+    (property "Value" "wire" (id 1) (at 197.485 38.1 0))
     (property "Footprint" "Connector_PinHeader_2.54mm:PinHeader_1x01_P2.54mm_Vertical" (id 2) (at 196.85 40.64 0)
       (effects (font (size 1.27 1.27)) hide)
@@
     (in_bom yes) (on_board yes) (fields_autoplaced)
     (property "Reference" "RL1" (id 0) (at 215.83 49.5 90))
-    (property "Value" "RL1" (id 1) (at 215.83 52.04 90))
+    (property "Value" "RL" (id 1) (at 215.83 52.04 90))
     (property "Footprint" "Library:Panasonic_AQ-G_relay" (id 2) (at 219.64 63.47 0)
       (effects (font (size 1.27 1.27)) hide)
@@
     )
     (path "/ce0dbf7b-cd46-4dcb-89ff-d7c45c41cb27"
-      (reference "J4") (unit 1) (value "AC/N") (footprint "Connector_PinHeader_2.54mm:PinHeader_1x01_P2.54mm_Vertical")
+      (reference "J4") (unit 1) (value "wire") (footprint "Connector_PinHeader_2.54mm:PinHeader_1x01_P2.54mm_Vertical")
     )
     (path "/1d83a17d-bf7a-4f87-a295-e42a092793ee"
-      (reference "J5") (unit 1) (value "AC/L") (footprint "Connector_PinHeader_2.54mm:PinHeader_1x01_P2.54mm_Vertical")
+      (reference "J5") (unit 1) (value "wire") (footprint "Connector_PinHeader_2.54mm:PinHeader_1x01_P2.54mm_Vertical")
     )
     (path "/58a6b9b3-7c45-4082-80d8-cb22a1fd4263"
-      (reference "J6") (unit 1) (value "GND") (footprint "Connector_PinHeader_2.54mm:PinHeader_1x01_P2.54mm_Vertical")
+      (reference "J6") (unit 1) (value "wire") (footprint "Connector_PinHeader_2.54mm:PinHeader_1x01_P2.54mm_Vertical")
     )
     (path "/a0e94c56-f36a-497f-8fec-d0cf6acaaa5f"
-      (reference "J7") (unit 1) (value "5V") (footprint "Connector_PinHeader_2.54mm:PinHeader_1x01_P2.54mm_Vertical")
+      (reference "J7") (unit 1) (value "wire") (footprint "Connector_PinHeader_2.54mm:PinHeader_1x01_P2.54mm_Vertical")
     )
     (path "/706b063e-0d8f-4a51-90ba-78ac1fe2b45c"
@@
     )
     (path "/f27ae564-6571-4c5c-b8e8-9f9d010b4989"
-      (reference "RL1") (unit 1) (value "RL1") (footprint "Library:Panasonic_AQ-G_relay")
+      (reference "RL1") (unit 1) (value "RL") (footprint "Library:Panasonic_AQ-G_relay")
     )
     (path "/84a1bbb7-d858-47ec-a6c4-31ee625d38b1"
-      (reference "RL2") (unit 1) (value "RL2") (footprint "Library:Panasonic_AQ-G_relay")
+      (reference "RL2") (unit 1) (value "RL") (footprint "Library:Panasonic_AQ-G_relay")
     )
     (path "/774b0565-5bbf-4e29-8d1a-6015f7ad6631"
-      (reference "RL3") (unit 1) (value "RL3") (footprint "Library:Panasonic_AQ-G_relay")
+      (reference "RL3") (unit 1) (value "RL") (footprint "Library:Panasonic_AQ-G_relay")
     )
     (path "/571dc026-e79d-4541-a087-94909fbad973"
-      (reference "RL4") (unit 1) (value "RL4") (footprint "Library:Panasonic_AQ-G_relay")
+      (reference "RL4") (unit 1) (value "RL") (footprint "Library:Panasonic_AQ-G_relay")
     )
     (path "/1126fcf5-4d18-465f-92e2-ec4926402081"
-      (reference "RL5") (unit 1) (value "RL4") (footprint "Library:Panasonic_AQ-G_relay")
+      (reference "RL5") (unit 1) (value "RL") (footprint "Library:Panasonic_AQ-G_relay")
     )
     (path "/39f3ed5b-b1fc-4815-892d-1e87701accc5"
